File: PCB_design/audio_mixer_kicad/power.kicad_sch (KiCad schematic)
At the start: 84 parts, among them Q1 CSD19537Q3, U3 TPS7A2033PDBVR, U4 TPS563209DDCR, U5 TLV62569ADRLT, U6 LM5155DSSR, U7 ADP5070AREZ, U8 TPS7A4901DGNR, U9 TPS7A3001DGNR

Commit message: Reannotate and add passives for Y1
Parts:
- renumbered C9 to C10, C10 to C11, C11 to C12, C12 to C13, C13 to C14, C14 to C15, C15 to C16, C16 to C17, C17 to C18, C18 to C19, C1 to C2, C19 to C20, C20 to C21, C21 to C22, C22 to C23, C23 to C24, C24 to C25, C25 to C26, C26 to C27, C27 to C28, C28 to C29, C2 to C3, C29 to C30, C30 to C31, C31 to C32, C32 to C33, C33 to C34, C34 to C35, C35 to C36, C36 to C37, C37 to C38, C38 to C39, C3 to C4, C39 to C40, C40 to C41, C41 to C42, C4 to C5, C5 to C6, C6 to C7, C7 to C8, C8 to C9, R8 to R10, R9 to R11, R10 to R12, R11 to R13, R12 to R14, R13 to R15, R14 to R16, R15 to R17, R16 to R18, R17 to R19, R18 to R20, R19 to R21, R20 to R22, R21 to R23, R22 to R24, R23 to R25, R24 to R26, R25 to R27, R26 to R28, R27 to R29, R28 to R30, R29 to R31, R7 to R9
