File: PCB_design/audio_mixer_kicad/power.kicad_sch (KiCad schematic)
At the start: 84 parts, among them Q1 CSD19537Q3, U3 TPS7A2033PDBVR, U4 TPS563209DDCR, U5 TLV62569ADRLT, U6 LM5155DSSR, U7 ADP5070AREZ, U8 TPS7A4901DGNR, U9 TPS7A3001DGNR

Commit message: Assign footprints
Parts:
- C10, C11, C12, C13, C14, C15, C16, C17, C18, C19, C2, C20, C21, C22, C23, C24, C25, C26, C27, C28, C29, C3, C30, C31, C32, C33, C34, C35, C36, C37, C38, C39, C4, C40, C41, C42, C5, C6, C7, C8, C9: footprint (none) -> Capacitor_SMD:C_1206_3216Metric_Pad1.33x1.80mm_HandSolder
- D3: footprint (none) -> SS2PH10:DO-220AA_SS2PH10-M3&slash_84A_VIS
- D4, D5: footprint (none) -> B0540W:SOD123_DIO-M
- FB1, FB2, FB3, L1, L2, L3, L4, L5, L6: footprint (none) -> Inductor_SMD:L_1206_3216Metric_Pad1.22x1.90mm_HandSolder
- R10, R11, R12, R13, R14, R15, R16, R17, R18, R19, R20, R21, R22, R23, R24, R25, R26, R27, R28, R29, R30, R31, R9: footprint (none) -> Resistor_SMD:R_1206_3216Metric_Pad1.30x1.75mm_HandSolder
- U3: footprint DBV0005A-IPC_A -> TPS7A2033:DBV0005A-IPC_A
- U4: footprint DDC0006A -> TPS563209:DDC0006A
- U5: footprint DRL0006A -> TLV62569:DRL0006A
- U6: footprint DSS0012B -> LM5155:DSS0012B
- U8: footprint DGN8_1P89X1P57 -> TPA7A49:DGN8_1P89X1P57
- U9: footprint DGN8_1P89X1P57 -> TPS7A30:DGN8_1P89X1P57
