File: PCB_design/audio_mixer_kicad/audio_mixer_kicad.kicad_pcb (KiCad board)
At the start: 4 copper layers, 0 parts

Commit message: Assign footprints
Parts:
- added C1: 0.1u, Capacitor_SMD:C_1206_3216Metric_Pad1.33x1.80mm_HandSolder, F.Cu at (106.2, 56.9)
- added C10: 100n, Capacitor_SMD:C_1206_3216Metric_Pad1.33x1.80mm_HandSolder, F.Cu at (121.5, 13.5)
- added C100: 0.1u, Capacitor_SMD:C_1206_3216Metric_Pad1.33x1.80mm_HandSolder, F.Cu at (163.9, 95.4)
- added C101: 2.2n, Capacitor_SMD:C_1206_3216Metric_Pad1.33x1.80mm_HandSolder, F.Cu at (163.9, 98.8)
- added C102: 10u, Capacitor_SMD:C_1206_3216Metric_Pad1.33x1.80mm_HandSolder, F.Cu at (163.9, 102.1)
- added C103: 0.1u, Capacitor_SMD:C_1206_3216Metric_Pad1.33x1.80mm_HandSolder, F.Cu at (163.9, 105.5)
- added C104: 2.2n, Capacitor_SMD:C_1206_3216Metric_Pad1.33x1.80mm_HandSolder, F.Cu at (163.9, 108.8)
- added C105: 1u, Capacitor_SMD:C_1206_3216Metric_Pad1.33x1.80mm_HandSolder, F.Cu at (163.9, 112.2)
- added C106: 2.2n, Capacitor_SMD:C_1206_3216Metric_Pad1.33x1.80mm_HandSolder, F.Cu at (169.9, 95.4)
- added C107: 10u, Capacitor_SMD:C_1206_3216Metric_Pad1.33x1.80mm_HandSolder, F.Cu at (169.9, 98.8)
- added C108: 0.1u, Capacitor_SMD:C_1206_3216Metric_Pad1.33x1.80mm_HandSolder, F.Cu at (169.9, 102.1)
- added C109: 10u, Capacitor_SMD:C_1206_3216Metric_Pad1.33x1.80mm_HandSolder, F.Cu at (169.9, 105.5)
- added C11: 10u, Capacitor_SMD:C_1206_3216Metric_Pad1.33x1.80mm_HandSolder, F.Cu at (121.5, 16.9)
- added C110: 0.1u, Capacitor_SMD:C_1206_3216Metric_Pad1.33x1.80mm_HandSolder, F.Cu at (169.9, 108.8)
- added C111: 2.2n, Capacitor_SMD:C_1206_3216Metric_Pad1.33x1.80mm_HandSolder, F.Cu at (37.0, 163.3)
- added C112: 2.2n, Capacitor_SMD:C_1206_3216Metric_Pad1.33x1.80mm_HandSolder, F.Cu at (37.0, 166.7)
- added C113: 2.2n, Capacitor_SMD:C_1206_3216Metric_Pad1.33x1.80mm_HandSolder, F.Cu at (37.0, 170.0)
- added C114: 2.2n, Capacitor_SMD:C_1206_3216Metric_Pad1.33x1.80mm_HandSolder, F.Cu at (37.0, 173.4)
- added C115: 2.2n, Capacitor_SMD:C_1206_3216Metric_Pad1.33x1.80mm_HandSolder, F.Cu at (37.0, 176.7)
- added C116: 10u, Capacitor_SMD:C_1206_3216Metric_Pad1.33x1.80mm_HandSolder, F.Cu at (37.0, 180.1)
- added C117: 0.1u, Capacitor_SMD:C_1206_3216Metric_Pad1.33x1.80mm_HandSolder, F.Cu at (43.0, 163.3)
- added C118: 2.2n, Capacitor_SMD:C_1206_3216Metric_Pad1.33x1.80mm_HandSolder, F.Cu at (43.0, 166.7)
- added C119: 10u, Capacitor_SMD:C_1206_3216Metric_Pad1.33x1.80mm_HandSolder, F.Cu at (43.0, 170.0)
- added C12: 49.755n, Capacitor_SMD:C_1206_3216Metric_Pad1.33x1.80mm_HandSolder, F.Cu at (121.5, 20.2)
- added C120: 0.1u, Capacitor_SMD:C_1206_3216Metric_Pad1.33x1.80mm_HandSolder, F.Cu at (43.0, 173.4)
- added C121: 2.2n, Capacitor_SMD:C_1206_3216Metric_Pad1.33x1.80mm_HandSolder, F.Cu at (43.0, 176.7)
- added C122: 1u, Capacitor_SMD:C_1206_3216Metric_Pad1.33x1.80mm_HandSolder, F.Cu at (43.0, 180.1)
- added C123: 2.2n, Capacitor_SMD:C_1206_3216Metric_Pad1.33x1.80mm_HandSolder, F.Cu at (49.0, 163.3)
- added C124: 10u, Capacitor_SMD:C_1206_3216Metric_Pad1.33x1.80mm_HandSolder, F.Cu at (49.0, 166.7)
- added C125: 0.1u, Capacitor_SMD:C_1206_3216Metric_Pad1.33x1.80mm_HandSolder, F.Cu at (49.0, 170.0)
- added C126: 10u, Capacitor_SMD:C_1206_3216Metric_Pad1.33x1.80mm_HandSolder, F.Cu at (49.0, 173.4)
- added C127: 0.1u, Capacitor_SMD:C_1206_3216Metric_Pad1.33x1.80mm_HandSolder, F.Cu at (49.0, 176.7)
- added C128: 2.2n, Capacitor_SMD:C_1206_3216Metric_Pad1.33x1.80mm_HandSolder, F.Cu at (10.5, 163.3)
- added C129: 2.2n, Capacitor_SMD:C_1206_3216Metric_Pad1.33x1.80mm_HandSolder, F.Cu at (10.5, 166.7)
- added C13: 10u, Capacitor_SMD:C_1206_3216Metric_Pad1.33x1.80mm_HandSolder, F.Cu at (121.5, 23.6)
- added C130: 2.2n, Capacitor_SMD:C_1206_3216Metric_Pad1.33x1.80mm_HandSolder, F.Cu at (10.5, 170.0)
- added C131: 2.2n, Capacitor_SMD:C_1206_3216Metric_Pad1.33x1.80mm_HandSolder, F.Cu at (10.5, 173.4)
- added C132: 2.2n, Capacitor_SMD:C_1206_3216Metric_Pad1.33x1.80mm_HandSolder, F.Cu at (10.5, 176.7)
- added C133: 10u, Capacitor_SMD:C_1206_3216Metric_Pad1.33x1.80mm_HandSolder, F.Cu at (10.5, 180.1)
- added C134: 0.1u, Capacitor_SMD:C_1206_3216Metric_Pad1.33x1.80mm_HandSolder, F.Cu at (16.5, 163.3)
- added C135: 2.2n, Capacitor_SMD:C_1206_3216Metric_Pad1.33x1.80mm_HandSolder, F.Cu at (16.5, 166.7)
- added C136: 10u, Capacitor_SMD:C_1206_3216Metric_Pad1.33x1.80mm_HandSolder, F.Cu at (16.5, 170.0)
- added C137: 0.1u, Capacitor_SMD:C_1206_3216Metric_Pad1.33x1.80mm_HandSolder, F.Cu at (16.5, 173.4)
- added C138: 2.2n, Capacitor_SMD:C_1206_3216Metric_Pad1.33x1.80mm_HandSolder, F.Cu at (16.5, 176.7)
- added C139: 1u, Capacitor_SMD:C_1206_3216Metric_Pad1.33x1.80mm_HandSolder, F.Cu at (16.5, 180.1)
- added C14: 10u, Capacitor_SMD:C_1206_3216Metric_Pad1.33x1.80mm_HandSolder, F.Cu at (121.5, 26.9)
- added C140: 2.2n, Capacitor_SMD:C_1206_3216Metric_Pad1.33x1.80mm_HandSolder, F.Cu at (22.5, 163.3)
- added C141: 10u, Capacitor_SMD:C_1206_3216Metric_Pad1.33x1.80mm_HandSolder, F.Cu at (22.5, 166.7)
- added C142: 0.1u, Capacitor_SMD:C_1206_3216Metric_Pad1.33x1.80mm_HandSolder, F.Cu at (22.5, 170.0)
- added C143: 10u, Capacitor_SMD:C_1206_3216Metric_Pad1.33x1.80mm_HandSolder, F.Cu at (22.5, 173.4)
- added C144: 0.1u, Capacitor_SMD:C_1206_3216Metric_Pad1.33x1.80mm_HandSolder, F.Cu at (22.5, 176.7)
- added C145: 2.2n, Capacitor_SMD:C_1206_3216Metric_Pad1.33x1.80mm_HandSolder, F.Cu at (84.2, 163.3)
- added C146: 2.2n, Capacitor_SMD:C_1206_3216Metric_Pad1.33x1.80mm_HandSolder, F.Cu at (84.2, 166.7)
- added C147: 2.2n, Capacitor_SMD:C_1206_3216Metric_Pad1.33x1.80mm_HandSolder, F.Cu at (84.2, 170.0)
- added C148: 2.2n, Capacitor_SMD:C_1206_3216Metric_Pad1.33x1.80mm_HandSolder, F.Cu at (84.2, 173.4)
- added C149: 2.2n, Capacitor_SMD:C_1206_3216Metric_Pad1.33x1.80mm_HandSolder, F.Cu at (84.2, 176.7)
- added C15: 470p, Capacitor_SMD:C_1206_3216Metric_Pad1.33x1.80mm_HandSolder, F.Cu at (121.5, 30.3)
- added C150: 10u, Capacitor_SMD:C_1206_3216Metric_Pad1.33x1.80mm_HandSolder, F.Cu at (84.2, 180.1)
- added C151: 0.1u, Capacitor_SMD:C_1206_3216Metric_Pad1.33x1.80mm_HandSolder, F.Cu at (90.2, 163.3)
- added C152: 2.2n, Capacitor_SMD:C_1206_3216Metric_Pad1.33x1.80mm_HandSolder, F.Cu at (90.2, 166.7)
- added C153: 10u, Capacitor_SMD:C_1206_3216Metric_Pad1.33x1.80mm_HandSolder, F.Cu at (90.2, 170.0)
- added C154: 0.1u, Capacitor_SMD:C_1206_3216Metric_Pad1.33x1.80mm_HandSolder, F.Cu at (90.2, 173.4)
- added C155: 2.2n, Capacitor_SMD:C_1206_3216Metric_Pad1.33x1.80mm_HandSolder, F.Cu at (90.2, 176.7)
- added C156: 1u, Capacitor_SMD:C_1206_3216Metric_Pad1.33x1.80mm_HandSolder, F.Cu at (90.2, 180.1)
- added C157: 2.2n, Capacitor_SMD:C_1206_3216Metric_Pad1.33x1.80mm_HandSolder, F.Cu at (96.2, 163.3)
- added C158: 10u, Capacitor_SMD:C_1206_3216Metric_Pad1.33x1.80mm_HandSolder, F.Cu at (96.2, 166.7)
- added C159: 0.1u, Capacitor_SMD:C_1206_3216Metric_Pad1.33x1.80mm_HandSolder, F.Cu at (96.2, 170.0)
- added C16: 12p, Capacitor_SMD:C_1206_3216Metric_Pad1.33x1.80mm_HandSolder, F.Cu at (127.5, 10.2)
- added C160: 10u, Capacitor_SMD:C_1206_3216Metric_Pad1.33x1.80mm_HandSolder, F.Cu at (96.2, 173.4)
- added C161: 0.1u, Capacitor_SMD:C_1206_3216Metric_Pad1.33x1.80mm_HandSolder, F.Cu at (96.2, 176.7)
- added C162: 2.2n, Capacitor_SMD:C_1206_3216Metric_Pad1.33x1.80mm_HandSolder, F.Cu at (137.1, 163.3)
- added C163: 2.2n, Capacitor_SMD:C_1206_3216Metric_Pad1.33x1.80mm_HandSolder, F.Cu at (137.1, 166.7)
- added C164: 2.2n, Capacitor_SMD:C_1206_3216Metric_Pad1.33x1.80mm_HandSolder, F.Cu at (137.1, 170.0)
- added C165: 2.2n, Capacitor_SMD:C_1206_3216Metric_Pad1.33x1.80mm_HandSolder, F.Cu at (137.1, 173.4)
- added C166: 2.2n, Capacitor_SMD:C_1206_3216Metric_Pad1.33x1.80mm_HandSolder, F.Cu at (137.1, 176.7)
- added C167: 10u, Capacitor_SMD:C_1206_3216Metric_Pad1.33x1.80mm_HandSolder, F.Cu at (137.1, 180.1)
- added C168: 0.1u, Capacitor_SMD:C_1206_3216Metric_Pad1.33x1.80mm_HandSolder, F.Cu at (143.1, 163.3)
- added C169: 2.2n, Capacitor_SMD:C_1206_3216Metric_Pad1.33x1.80mm_HandSolder, F.Cu at (143.1, 166.7)
- added C17: 1u, Capacitor_SMD:C_1206_3216Metric_Pad1.33x1.80mm_HandSolder, F.Cu at (127.5, 13.5)
- added C170: 10u, Capacitor_SMD:C_1206_3216Metric_Pad1.33x1.80mm_HandSolder, F.Cu at (143.1, 170.0)
- added C171: 0.1u, Capacitor_SMD:C_1206_3216Metric_Pad1.33x1.80mm_HandSolder, F.Cu at (143.1, 173.4)
- added C172: 2.2n, Capacitor_SMD:C_1206_3216Metric_Pad1.33x1.80mm_HandSolder, F.Cu at (143.1, 176.7)
- added C173: 1u, Capacitor_SMD:C_1206_3216Metric_Pad1.33x1.80mm_HandSolder, F.Cu at (143.1, 180.1)
- added C174: 2.2n, Capacitor_SMD:C_1206_3216Metric_Pad1.33x1.80mm_HandSolder, F.Cu at (149.1, 163.3)
- added C175: 10u, Capacitor_SMD:C_1206_3216Metric_Pad1.33x1.80mm_HandSolder, F.Cu at (149.1, 166.7)
- added C176: 0.1u, Capacitor_SMD:C_1206_3216Metric_Pad1.33x1.80mm_HandSolder, F.Cu at (149.1, 170.0)
- added C177: 10u, Capacitor_SMD:C_1206_3216Metric_Pad1.33x1.80mm_HandSolder, F.Cu at (149.1, 173.4)
- added C178: 0.1u, Capacitor_SMD:C_1206_3216Metric_Pad1.33x1.80mm_HandSolder, F.Cu at (149.1, 176.7)
- added C179: 0.1u 16V, Capacitor_SMD:C_1206_3216Metric_Pad1.33x1.80mm_HandSolder, F.Cu at (163.6, 163.3)
- added C18: 1u, Capacitor_SMD:C_1206_3216Metric_Pad1.33x1.80mm_HandSolder, F.Cu at (127.5, 16.9)
- added C180: 0.1u 16V, Capacitor_SMD:C_1206_3216Metric_Pad1.33x1.80mm_HandSolder, F.Cu at (163.6, 166.7)
- added C181: 10u 16V, Capacitor_SMD:C_1206_3216Metric_Pad1.33x1.80mm_HandSolder, F.Cu at (163.6, 170.0)
- added C182: 10u 16V, Capacitor_SMD:C_1206_3216Metric_Pad1.33x1.80mm_HandSolder, F.Cu at (163.6, 173.4)
- added C183: 1u 16V, Capacitor_SMD:C_1206_3216Metric_Pad1.33x1.80mm_HandSolder, F.Cu at (163.6, 176.7)
- added C184: 4.7n, Capacitor_SMD:C_1206_3216Metric_Pad1.33x1.80mm_HandSolder, F.Cu at (163.6, 180.1)
- added C185: 4.7n, Capacitor_SMD:C_1206_3216Metric_Pad1.33x1.80mm_HandSolder, F.Cu at (163.6, 183.4)
- added C186: 0.1u 16V, Capacitor_SMD:C_1206_3216Metric_Pad1.33x1.80mm_HandSolder, F.Cu at (163.6, 186.8)
- added C187: 10u 16V, Capacitor_SMD:C_1206_3216Metric_Pad1.33x1.80mm_HandSolder, F.Cu at (163.6, 190.1)
- added C188: 0.1u 16V, Capacitor_SMD:C_1206_3216Metric_Pad1.33x1.80mm_HandSolder, F.Cu at (63.4, 163.3)
- added C189: 0.1u 16V, Capacitor_SMD:C_1206_3216Metric_Pad1.33x1.80mm_HandSolder, F.Cu at (63.4, 166.7)
- added C19: 1u, Capacitor_SMD:C_1206_3216Metric_Pad1.33x1.80mm_HandSolder, F.Cu at (127.5, 20.2)
- added C190: 10u 16V, Capacitor_SMD:C_1206_3216Metric_Pad1.33x1.80mm_HandSolder, F.Cu at (63.4, 170.0)
- added C191: 10u 16V, Capacitor_SMD:C_1206_3216Metric_Pad1.33x1.80mm_HandSolder, F.Cu at (63.4, 173.4)
- added C192: 1u 16V, Capacitor_SMD:C_1206_3216Metric_Pad1.33x1.80mm_HandSolder, F.Cu at (63.4, 176.7)
- added C193: 4.7n, Capacitor_SMD:C_1206_3216Metric_Pad1.33x1.80mm_HandSolder, F.Cu at (63.4, 180.1)
- added C194: 4.7n, Capacitor_SMD:C_1206_3216Metric_Pad1.33x1.80mm_HandSolder, F.Cu at (63.4, 183.4)
- added C195: 0.1u 16V, Capacitor_SMD:C_1206_3216Metric_Pad1.33x1.80mm_HandSolder, F.Cu at (63.4, 186.8)
- added C196: 10u 16V, Capacitor_SMD:C_1206_3216Metric_Pad1.33x1.80mm_HandSolder, F.Cu at (63.4, 190.1)
- added C197: 100n, Capacitor_SMD:C_1206_3216Metric_Pad1.33x1.80mm_HandSolder, F.Cu at (168.3, 36.1)
- added C198: 100n, Capacitor_SMD:C_1206_3216Metric_Pad1.33x1.80mm_HandSolder, F.Cu at (168.3, 39.4)
- added C199: 100n, Capacitor_SMD:C_1206_3216Metric_Pad1.33x1.80mm_HandSolder, F.Cu at (168.3, 42.8)
- added C2: 10u, Capacitor_SMD:C_1206_3216Metric_Pad1.33x1.80mm_HandSolder, F.Cu at (115.5, 10.2)
- added C20: 100n, Capacitor_SMD:C_1206_3216Metric_Pad1.33x1.80mm_HandSolder, F.Cu at (127.5, 23.6)
- added C200: 100p, Capacitor_SMD:C_1206_3216Metric_Pad1.33x1.80mm_HandSolder, F.Cu at (168.3, 46.1)
- added C201: 100p, Capacitor_SMD:C_1206_3216Metric_Pad1.33x1.80mm_HandSolder, F.Cu at (168.3, 49.5)
- added C202: 100n, Capacitor_SMD:C_1206_3216Metric_Pad1.33x1.80mm_HandSolder, F.Cu at (168.3, 10.2)
- added C203: 100n, Capacitor_SMD:C_1206_3216Metric_Pad1.33x1.80mm_HandSolder, F.Cu at (168.3, 13.5)
- added C204: 100n, Capacitor_SMD:C_1206_3216Metric_Pad1.33x1.80mm_HandSolder, F.Cu at (168.3, 16.9)
- added C205: 100p, Capacitor_SMD:C_1206_3216Metric_Pad1.33x1.80mm_HandSolder, F.Cu at (168.3, 20.2)
- added C206: 100p, Capacitor_SMD:C_1206_3216Metric_Pad1.33x1.80mm_HandSolder, F.Cu at (168.3, 23.6)
- added C207: 100n, Capacitor_SMD:C_1206_3216Metric_Pad1.33x1.80mm_HandSolder, F.Cu at (168.3, 62.0)
- added C208: 100n, Capacitor_SMD:C_1206_3216Metric_Pad1.33x1.80mm_HandSolder, F.Cu at (168.3, 65.3)
- added C209: 100n, Capacitor_SMD:C_1206_3216Metric_Pad1.33x1.80mm_HandSolder, F.Cu at (168.3, 68.7)
- added C21: 6.8n, Capacitor_SMD:C_1206_3216Metric_Pad1.33x1.80mm_HandSolder, F.Cu at (127.5, 26.9)
- added C210: 100p, Capacitor_SMD:C_1206_3216Metric_Pad1.33x1.80mm_HandSolder, F.Cu at (168.3, 72.0)
- added C211: 100p, Capacitor_SMD:C_1206_3216Metric_Pad1.33x1.80mm_HandSolder, F.Cu at (168.3, 75.4)
- added C212: 100n, Capacitor_SMD:C_1206_3216Metric_Pad1.33x1.80mm_HandSolder, F.Cu at (129.4, 66.7)
- added C213: 100n, Capacitor_SMD:C_1206_3216Metric_Pad1.33x1.80mm_HandSolder, F.Cu at (129.4, 70.0)
- added C214: 100n, Capacitor_SMD:C_1206_3216Metric_Pad1.33x1.80mm_HandSolder, F.Cu at (129.4, 73.4)
- added C215: 100p, Capacitor_SMD:C_1206_3216Metric_Pad1.33x1.80mm_HandSolder, F.Cu at (129.4, 76.7)
- added C216: 100p, Capacitor_SMD:C_1206_3216Metric_Pad1.33x1.80mm_HandSolder, F.Cu at (129.4, 80.1)
- added C217: 47u 63V, Capacitor_SMD:C_1206_3216Metric_Pad1.33x1.80mm_HandSolder, F.Cu at (52.2, 95.4)
- added C218: 47u 63V, Capacitor_SMD:C_1206_3216Metric_Pad1.33x1.80mm_HandSolder, F.Cu at (52.2, 98.8)
- added C219: 47u 63V, Capacitor_SMD:C_1206_3216Metric_Pad1.33x1.80mm_HandSolder, F.Cu at (52.2, 102.1)
- added C22: 10u, Capacitor_SMD:C_1206_3216Metric_Pad1.33x1.80mm_HandSolder, F.Cu at (127.5, 30.3)
- added C220: 47u 63V, Capacitor_SMD:C_1206_3216Metric_Pad1.33x1.80mm_HandSolder, F.Cu at (52.2, 105.5)
- added C221: 47u 63V, Capacitor_SMD:C_1206_3216Metric_Pad1.33x1.80mm_HandSolder, F.Cu at (52.2, 108.8)
- added C222: 47u 63V, Capacitor_SMD:C_1206_3216Metric_Pad1.33x1.80mm_HandSolder, F.Cu at (52.2, 112.2)
- added C223: 47u 63V, Capacitor_SMD:C_1206_3216Metric_Pad1.33x1.80mm_HandSolder, F.Cu at (52.2, 115.5)
- added C224: 47u 63V, Capacitor_SMD:C_1206_3216Metric_Pad1.33x1.80mm_HandSolder, F.Cu at (52.2, 118.9)
- added C225: 47u 63V, Capacitor_SMD:C_1206_3216Metric_Pad1.33x1.80mm_HandSolder, F.Cu at (52.2, 122.2)
- added C226: 47u 63V, Capacitor_SMD:C_1206_3216Metric_Pad1.33x1.80mm_HandSolder, F.Cu at (52.2, 125.6)
- added C227: 47u 63V, Capacitor_SMD:C_1206_3216Metric_Pad1.33x1.80mm_HandSolder, F.Cu at (58.2, 95.4)
- added C228: 47u 63V, Capacitor_SMD:C_1206_3216Metric_Pad1.33x1.80mm_HandSolder, F.Cu at (58.2, 98.8)
- added C229: 47u 63V, Capacitor_SMD:C_1206_3216Metric_Pad1.33x1.80mm_HandSolder, F.Cu at (58.2, 102.1)
- added C23: 47p, Capacitor_SMD:C_1206_3216Metric_Pad1.33x1.80mm_HandSolder, F.Cu at (133.5, 10.2)
- added C230: 47u 63V, Capacitor_SMD:C_1206_3216Metric_Pad1.33x1.80mm_HandSolder, F.Cu at (58.2, 105.5)
- added C231: 47u 63V, Capacitor_SMD:C_1206_3216Metric_Pad1.33x1.80mm_HandSolder, F.Cu at (58.2, 108.8)
- added C232: 47u 63V, Capacitor_SMD:C_1206_3216Metric_Pad1.33x1.80mm_HandSolder, F.Cu at (58.2, 112.2)
- added C233: 10u, Capacitor_SMD:C_1206_3216Metric_Pad1.33x1.80mm_HandSolder, F.Cu at (58.2, 115.5)
- added C234: 10u, Capacitor_SMD:C_1206_3216Metric_Pad1.33x1.80mm_HandSolder, F.Cu at (58.2, 118.9)
- added C235: 10u, Capacitor_SMD:C_1206_3216Metric_Pad1.33x1.80mm_HandSolder, F.Cu at (58.2, 122.2)
- added C236: 10u, Capacitor_SMD:C_1206_3216Metric_Pad1.33x1.80mm_HandSolder, F.Cu at (58.2, 125.6)
- added C237: 10u, Capacitor_SMD:C_1206_3216Metric_Pad1.33x1.80mm_HandSolder, F.Cu at (64.2, 95.4)
- added C238: 10u, Capacitor_SMD:C_1206_3216Metric_Pad1.33x1.80mm_HandSolder, F.Cu at (64.2, 98.8)
- added C239: 10u, Capacitor_SMD:C_1206_3216Metric_Pad1.33x1.80mm_HandSolder, F.Cu at (64.2, 102.1)
- added C24: 22u, Capacitor_SMD:C_1206_3216Metric_Pad1.33x1.80mm_HandSolder, F.Cu at (133.5, 13.5)
- added C240: 10u, Capacitor_SMD:C_1206_3216Metric_Pad1.33x1.80mm_HandSolder, F.Cu at (64.2, 105.5)
- added C241: 47u 63V, Capacitor_SMD:C_1206_3216Metric_Pad1.33x1.80mm_HandSolder, F.Cu at (64.2, 108.8)
- added C242: 47u 63V, Capacitor_SMD:C_1206_3216Metric_Pad1.33x1.80mm_HandSolder, F.Cu at (64.2, 112.2)
- added C243: 47u 63V, Capacitor_SMD:C_1206_3216Metric_Pad1.33x1.80mm_HandSolder, F.Cu at (64.2, 115.5)
- added C244: 47u 63V, Capacitor_SMD:C_1206_3216Metric_Pad1.33x1.80mm_HandSolder, F.Cu at (64.2, 118.9)
- added C245: 47u 63V, Capacitor_SMD:C_1206_3216Metric_Pad1.33x1.80mm_HandSolder, F.Cu at (64.2, 122.2)
- added C246: 47u 63V, Capacitor_SMD:C_1206_3216Metric_Pad1.33x1.80mm_HandSolder, F.Cu at (64.2, 125.6)
- added C247: 47u 63V, Capacitor_SMD:C_1206_3216Metric_Pad1.33x1.80mm_HandSolder, F.Cu at (70.2, 95.4)
- added C248: 47u 63V, Capacitor_SMD:C_1206_3216Metric_Pad1.33x1.80mm_HandSolder, F.Cu at (70.2, 98.8)
- added C249: 47u 63V, Capacitor_SMD:C_1206_3216Metric_Pad1.33x1.80mm_HandSolder, F.Cu at (70.2, 102.1)
- added C25: 22u, Capacitor_SMD:C_1206_3216Metric_Pad1.33x1.80mm_HandSolder, F.Cu at (133.5, 16.9)
- added C250: 47u 63V, Capacitor_SMD:C_1206_3216Metric_Pad1.33x1.80mm_HandSolder, F.Cu at (70.2, 105.5)
- added C251: 47u 63V, Capacitor_SMD:C_1206_3216Metric_Pad1.33x1.80mm_HandSolder, F.Cu at (70.2, 108.8)
- added C252: 47u 63V, Capacitor_SMD:C_1206_3216Metric_Pad1.33x1.80mm_HandSolder, F.Cu at (70.2, 112.2)
- added C253: 47u 63V, Capacitor_SMD:C_1206_3216Metric_Pad1.33x1.80mm_HandSolder, F.Cu at (70.2, 115.5)
- added C254: 47u 63V, Capacitor_SMD:C_1206_3216Metric_Pad1.33x1.80mm_HandSolder, F.Cu at (70.2, 118.9)
- added C255: 47u 63V, Capacitor_SMD:C_1206_3216Metric_Pad1.33x1.80mm_HandSolder, F.Cu at (70.2, 122.2)
- added C256: 47u 63V, Capacitor_SMD:C_1206_3216Metric_Pad1.33x1.80mm_HandSolder, F.Cu at (70.2, 125.6)
- added C257: 10u, Capacitor_SMD:C_1206_3216Metric_Pad1.33x1.80mm_HandSolder, F.Cu at (76.2, 95.4)
- added C258: 10u, Capacitor_SMD:C_1206_3216Metric_Pad1.33x1.80mm_HandSolder, F.Cu at (76.2, 98.8)
- added C259: 10u, Capacitor_SMD:C_1206_3216Metric_Pad1.33x1.80mm_HandSolder, F.Cu at (76.2, 102.1)
- added C26: 49.755n, Capacitor_SMD:C_1206_3216Metric_Pad1.33x1.80mm_HandSolder, F.Cu at (133.5, 20.2)
- added C260: 10u, Capacitor_SMD:C_1206_3216Metric_Pad1.33x1.80mm_HandSolder, F.Cu at (76.2, 105.5)
- added C261: 10u, Capacitor_SMD:C_1206_3216Metric_Pad1.33x1.80mm_HandSolder, F.Cu at (76.2, 108.8)
- added C262: 10u, Capacitor_SMD:C_1206_3216Metric_Pad1.33x1.80mm_HandSolder, F.Cu at (76.2, 112.2)
- added C263: 10u, Capacitor_SMD:C_1206_3216Metric_Pad1.33x1.80mm_HandSolder, F.Cu at (76.2, 115.5)
- added C264: 10u, Capacitor_SMD:C_1206_3216Metric_Pad1.33x1.80mm_HandSolder, F.Cu at (76.2, 118.9)
- added C265: 47u 63V, Capacitor_SMD:C_1206_3216Metric_Pad1.33x1.80mm_HandSolder, F.Cu at (125.9, 95.4)
- added C266: 47u 63V, Capacitor_SMD:C_1206_3216Metric_Pad1.33x1.80mm_HandSolder, F.Cu at (125.9, 98.8)
- added C267: 47u 63V, Capacitor_SMD:C_1206_3216Metric_Pad1.33x1.80mm_HandSolder, F.Cu at (125.9, 102.1)
- added C268: 47u 63V, Capacitor_SMD:C_1206_3216Metric_Pad1.33x1.80mm_HandSolder, F.Cu at (125.9, 105.5)
- added C269: 47u 63V, Capacitor_SMD:C_1206_3216Metric_Pad1.33x1.80mm_HandSolder, F.Cu at (125.9, 108.8)
- added C27: 22u, Capacitor_SMD:C_1206_3216Metric_Pad1.33x1.80mm_HandSolder, F.Cu at (133.5, 23.6)
- added C270: 47u 63V, Capacitor_SMD:C_1206_3216Metric_Pad1.33x1.80mm_HandSolder, F.Cu at (125.9, 112.2)
- added C271: 47u 63V, Capacitor_SMD:C_1206_3216Metric_Pad1.33x1.80mm_HandSolder, F.Cu at (125.9, 115.5)
- added C272: 47u 63V, Capacitor_SMD:C_1206_3216Metric_Pad1.33x1.80mm_HandSolder, F.Cu at (125.9, 118.9)
- added C273: 47u 63V, Capacitor_SMD:C_1206_3216Metric_Pad1.33x1.80mm_HandSolder, F.Cu at (125.9, 122.2)
- added C274: 47u 63V, Capacitor_SMD:C_1206_3216Metric_Pad1.33x1.80mm_HandSolder, F.Cu at (125.9, 125.6)
- added C275: 47u 63V, Capacitor_SMD:C_1206_3216Metric_Pad1.33x1.80mm_HandSolder, F.Cu at (131.9, 95.4)
- added C276: 47u 63V, Capacitor_SMD:C_1206_3216Metric_Pad1.33x1.80mm_HandSolder, F.Cu at (131.9, 98.8)
- added C277: 47u 63V, Capacitor_SMD:C_1206_3216Metric_Pad1.33x1.80mm_HandSolder, F.Cu at (131.9, 102.1)
- added C278: 47u 63V, Capacitor_SMD:C_1206_3216Metric_Pad1.33x1.80mm_HandSolder, F.Cu at (131.9, 105.5)
- added C279: 47u 63V, Capacitor_SMD:C_1206_3216Metric_Pad1.33x1.80mm_HandSolder, F.Cu at (131.9, 108.8)
- added C28: 1u, Capacitor_SMD:C_1206_3216Metric_Pad1.33x1.80mm_HandSolder, F.Cu at (133.5, 26.9)
- added C280: 47u 63V, Capacitor_SMD:C_1206_3216Metric_Pad1.33x1.80mm_HandSolder, F.Cu at (131.9, 112.2)
- added C281: 10u, Capacitor_SMD:C_1206_3216Metric_Pad1.33x1.80mm_HandSolder, F.Cu at (131.9, 115.5)
- added C282: 10u, Capacitor_SMD:C_1206_3216Metric_Pad1.33x1.80mm_HandSolder, F.Cu at (131.9, 118.9)
- added C283: 10u, Capacitor_SMD:C_1206_3216Metric_Pad1.33x1.80mm_HandSolder, F.Cu at (131.9, 122.2)
- added C284: 10u, Capacitor_SMD:C_1206_3216Metric_Pad1.33x1.80mm_HandSolder, F.Cu at (131.9, 125.6)
- added C285: 10u, Capacitor_SMD:C_1206_3216Metric_Pad1.33x1.80mm_HandSolder, F.Cu at (137.9, 95.4)
- added C286: 10u, Capacitor_SMD:C_1206_3216Metric_Pad1.33x1.80mm_HandSolder, F.Cu at (137.9, 98.8)
- added C287: 10u, Capacitor_SMD:C_1206_3216Metric_Pad1.33x1.80mm_HandSolder, F.Cu at (137.9, 102.1)
- added C288: 10u, Capacitor_SMD:C_1206_3216Metric_Pad1.33x1.80mm_HandSolder, F.Cu at (137.9, 105.5)
- added C289: 47u 63V, Capacitor_SMD:C_1206_3216Metric_Pad1.33x1.80mm_HandSolder, F.Cu at (137.9, 108.8)
- added C29: 1u, Capacitor_SMD:C_1206_3216Metric_Pad1.33x1.80mm_HandSolder, F.Cu at (133.5, 30.3)
- added C290: 47u 63V, Capacitor_SMD:C_1206_3216Metric_Pad1.33x1.80mm_HandSolder, F.Cu at (137.9, 112.2)
- added C291: 47u 63V, Capacitor_SMD:C_1206_3216Metric_Pad1.33x1.80mm_HandSolder, F.Cu at (137.9, 115.5)
- added C292: 47u 63V, Capacitor_SMD:C_1206_3216Metric_Pad1.33x1.80mm_HandSolder, F.Cu at (137.9, 118.9)
- added C293: 47u 63V, Capacitor_SMD:C_1206_3216Metric_Pad1.33x1.80mm_HandSolder, F.Cu at (137.9, 122.2)
- added C294: 47u 63V, Capacitor_SMD:C_1206_3216Metric_Pad1.33x1.80mm_HandSolder, F.Cu at (137.9, 125.6)
- added C295: 47u 63V, Capacitor_SMD:C_1206_3216Metric_Pad1.33x1.80mm_HandSolder, F.Cu at (143.9, 95.4)
- added C296: 47u 63V, Capacitor_SMD:C_1206_3216Metric_Pad1.33x1.80mm_HandSolder, F.Cu at (143.9, 98.8)
- added C297: 47u 63V, Capacitor_SMD:C_1206_3216Metric_Pad1.33x1.80mm_HandSolder, F.Cu at (143.9, 102.1)
- added C298: 47u 63V, Capacitor_SMD:C_1206_3216Metric_Pad1.33x1.80mm_HandSolder, F.Cu at (143.9, 105.5)
- added C299: 47u 63V, Capacitor_SMD:C_1206_3216Metric_Pad1.33x1.80mm_HandSolder, F.Cu at (143.9, 108.8)
- added C3: 10u, Capacitor_SMD:C_1206_3216Metric_Pad1.33x1.80mm_HandSolder, F.Cu at (115.5, 13.5)
- added C30: 4.7u, Capacitor_SMD:C_1206_3216Metric_Pad1.33x1.80mm_HandSolder, F.Cu at (139.5, 10.2)
- added C300: 47u 63V, Capacitor_SMD:C_1206_3216Metric_Pad1.33x1.80mm_HandSolder, F.Cu at (143.9, 112.2)
- added C301: 47u 63V, Capacitor_SMD:C_1206_3216Metric_Pad1.33x1.80mm_HandSolder, F.Cu at (143.9, 115.5)
- added C302: 47u 63V, Capacitor_SMD:C_1206_3216Metric_Pad1.33x1.80mm_HandSolder, F.Cu at (143.9, 118.9)
- added C303: 47u 63V, Capacitor_SMD:C_1206_3216Metric_Pad1.33x1.80mm_HandSolder, F.Cu at (143.9, 122.2)
- added C304: 47u 63V, Capacitor_SMD:C_1206_3216Metric_Pad1.33x1.80mm_HandSolder, F.Cu at (143.9, 125.6)
- added C305: 10u, Capacitor_SMD:C_1206_3216Metric_Pad1.33x1.80mm_HandSolder, F.Cu at (149.9, 95.4)
- added C306: 10u, Capacitor_SMD:C_1206_3216Metric_Pad1.33x1.80mm_HandSolder, F.Cu at (149.9, 98.8)
- added C307: 10u, Capacitor_SMD:C_1206_3216Metric_Pad1.33x1.80mm_HandSolder, F.Cu at (149.9, 102.1)
- added C308: 10u, Capacitor_SMD:C_1206_3216Metric_Pad1.33x1.80mm_HandSolder, F.Cu at (149.9, 105.5)
- added C309: 10u, Capacitor_SMD:C_1206_3216Metric_Pad1.33x1.80mm_HandSolder, F.Cu at (149.9, 108.8)
- added C31: 10n, Capacitor_SMD:C_1206_3216Metric_Pad1.33x1.80mm_HandSolder, F.Cu at (139.5, 13.5)
- added C310: 10u, Capacitor_SMD:C_1206_3216Metric_Pad1.33x1.80mm_HandSolder, F.Cu at (149.9, 112.2)
- added C311: 10u, Capacitor_SMD:C_1206_3216Metric_Pad1.33x1.80mm_HandSolder, F.Cu at (149.9, 115.5)
- added C312: 10u, Capacitor_SMD:C_1206_3216Metric_Pad1.33x1.80mm_HandSolder, F.Cu at (149.9, 118.9)
- added C32: 10n, Capacitor_SMD:C_1206_3216Metric_Pad1.33x1.80mm_HandSolder, F.Cu at (139.5, 16.9)
- added C33: 4.7u, Capacitor_SMD:C_1206_3216Metric_Pad1.33x1.80mm_HandSolder, F.Cu at (139.5, 20.2)
- added C34: 4.7u, Capacitor_SMD:C_1206_3216Metric_Pad1.33x1.80mm_HandSolder, F.Cu at (139.5, 23.6)
- added C35: 1u, Capacitor_SMD:C_1206_3216Metric_Pad1.33x1.80mm_HandSolder, F.Cu at (139.5, 26.9)
- added C36: 10u, Capacitor_SMD:C_1206_3216Metric_Pad1.33x1.80mm_HandSolder, F.Cu at (139.5, 30.3)
- added C37: 10u, Capacitor_SMD:C_1206_3216Metric_Pad1.33x1.80mm_HandSolder, F.Cu at (145.5, 10.2)
- added C38: 10u, Capacitor_SMD:C_1206_3216Metric_Pad1.33x1.80mm_HandSolder, F.Cu at (145.5, 13.5)
- added C39: 10u, Capacitor_SMD:C_1206_3216Metric_Pad1.33x1.80mm_HandSolder, F.Cu at (145.5, 16.9)
- added C4: 0.1u, Capacitor_SMD:C_1206_3216Metric_Pad1.33x1.80mm_HandSolder, F.Cu at (115.5, 16.9)
- added C40: 47u 63V, Capacitor_SMD:C_1206_3216Metric_Pad1.33x1.80mm_HandSolder, F.Cu at (145.5, 20.2)
- added C41: 0.1u, Capacitor_SMD:C_1206_3216Metric_Pad1.33x1.80mm_HandSolder, F.Cu at (145.5, 23.6)
- added C42: 0.1u, Capacitor_SMD:C_1206_3216Metric_Pad1.33x1.80mm_HandSolder, F.Cu at (145.5, 26.9)
- added C43: 2.2n, Capacitor_SMD:C_1206_3216Metric_Pad1.33x1.80mm_HandSolder, F.Cu at (157.9, 117.5)
- added C44: 2.2n, Capacitor_SMD:C_1206_3216Metric_Pad1.33x1.80mm_HandSolder, F.Cu at (157.9, 120.9)
- added C45: 2.2n, Capacitor_SMD:C_1206_3216Metric_Pad1.33x1.80mm_HandSolder, F.Cu at (157.9, 124.2)
- added C46: 2.2n, Capacitor_SMD:C_1206_3216Metric_Pad1.33x1.80mm_HandSolder, F.Cu at (157.9, 127.6)
- added C47: 2.2n, Capacitor_SMD:C_1206_3216Metric_Pad1.33x1.80mm_HandSolder, F.Cu at (157.9, 130.9)
- added C48: 10u, Capacitor_SMD:C_1206_3216Metric_Pad1.33x1.80mm_HandSolder, F.Cu at (157.9, 134.3)
- added C49: 0.1u, Capacitor_SMD:C_1206_3216Metric_Pad1.33x1.80mm_HandSolder, F.Cu at (163.9, 117.5)
- added C5: 10u, Capacitor_SMD:C_1206_3216Metric_Pad1.33x1.80mm_HandSolder, F.Cu at (115.5, 20.2)
- added C50: 2.2n, Capacitor_SMD:C_1206_3216Metric_Pad1.33x1.80mm_HandSolder, F.Cu at (163.9, 120.9)
- added C51: 10u, Capacitor_SMD:C_1206_3216Metric_Pad1.33x1.80mm_HandSolder, F.Cu at (163.9, 124.2)
- added C52: 0.1u, Capacitor_SMD:C_1206_3216Metric_Pad1.33x1.80mm_HandSolder, F.Cu at (163.9, 127.6)
- added C53: 2.2n, Capacitor_SMD:C_1206_3216Metric_Pad1.33x1.80mm_HandSolder, F.Cu at (163.9, 130.9)
- added C54: 1u, Capacitor_SMD:C_1206_3216Metric_Pad1.33x1.80mm_HandSolder, F.Cu at (163.9, 134.3)
- added C55: 2.2n, Capacitor_SMD:C_1206_3216Metric_Pad1.33x1.80mm_HandSolder, F.Cu at (169.9, 117.5)
- added C56: 10u, Capacitor_SMD:C_1206_3216Metric_Pad1.33x1.80mm_HandSolder, F.Cu at (169.9, 120.9)
- added C57: 0.1u, Capacitor_SMD:C_1206_3216Metric_Pad1.33x1.80mm_HandSolder, F.Cu at (169.9, 124.2)
- added C58: 10u, Capacitor_SMD:C_1206_3216Metric_Pad1.33x1.80mm_HandSolder, F.Cu at (169.9, 127.6)
- added C59: 0.1u, Capacitor_SMD:C_1206_3216Metric_Pad1.33x1.80mm_HandSolder, F.Cu at (169.9, 130.9)
- added C6: 10u, Capacitor_SMD:C_1206_3216Metric_Pad1.33x1.80mm_HandSolder, F.Cu at (115.5, 23.6)
- added C60: 2.2n, Capacitor_SMD:C_1206_3216Metric_Pad1.33x1.80mm_HandSolder, F.Cu at (110.7, 163.3)
- added C61: 2.2n, Capacitor_SMD:C_1206_3216Metric_Pad1.33x1.80mm_HandSolder, F.Cu at (110.7, 166.7)
- added C62: 2.2n, Capacitor_SMD:C_1206_3216Metric_Pad1.33x1.80mm_HandSolder, F.Cu at (110.7, 170.0)
- added C63: 2.2n, Capacitor_SMD:C_1206_3216Metric_Pad1.33x1.80mm_HandSolder, F.Cu at (110.7, 173.4)
- added C64: 2.2n, Capacitor_SMD:C_1206_3216Metric_Pad1.33x1.80mm_HandSolder, F.Cu at (110.7, 176.7)
- added C65: 10u, Capacitor_SMD:C_1206_3216Metric_Pad1.33x1.80mm_HandSolder, F.Cu at (110.7, 180.1)
- added C66: 0.1u, Capacitor_SMD:C_1206_3216Metric_Pad1.33x1.80mm_HandSolder, F.Cu at (116.7, 163.3)
- added C67: 2.2n, Capacitor_SMD:C_1206_3216Metric_Pad1.33x1.80mm_HandSolder, F.Cu at (116.7, 166.7)
- added C68: 10u, Capacitor_SMD:C_1206_3216Metric_Pad1.33x1.80mm_HandSolder, F.Cu at (116.7, 170.0)
- added C69: 0.1u, Capacitor_SMD:C_1206_3216Metric_Pad1.33x1.80mm_HandSolder, F.Cu at (116.7, 173.4)
- added C7: 4.7u, Capacitor_SMD:C_1206_3216Metric_Pad1.33x1.80mm_HandSolder, F.Cu at (115.5, 26.9)
- added C70: 2.2n, Capacitor_SMD:C_1206_3216Metric_Pad1.33x1.80mm_HandSolder, F.Cu at (116.7, 176.7)
- added C71: 1u, Capacitor_SMD:C_1206_3216Metric_Pad1.33x1.80mm_HandSolder, F.Cu at (116.7, 180.1)
- added C72: 2.2n, Capacitor_SMD:C_1206_3216Metric_Pad1.33x1.80mm_HandSolder, F.Cu at (122.7, 163.3)
- added C73: 10u, Capacitor_SMD:C_1206_3216Metric_Pad1.33x1.80mm_HandSolder, F.Cu at (122.7, 166.7)
- added C74: 0.1u, Capacitor_SMD:C_1206_3216Metric_Pad1.33x1.80mm_HandSolder, F.Cu at (122.7, 170.0)
- added C75: 10u, Capacitor_SMD:C_1206_3216Metric_Pad1.33x1.80mm_HandSolder, F.Cu at (122.7, 173.4)
- added C76: 0.1u, Capacitor_SMD:C_1206_3216Metric_Pad1.33x1.80mm_HandSolder, F.Cu at (122.7, 176.7)
- added C77: 2.2n, Capacitor_SMD:C_1206_3216Metric_Pad1.33x1.80mm_HandSolder, F.Cu at (157.9, 139.6)
- added C78: 2.2n, Capacitor_SMD:C_1206_3216Metric_Pad1.33x1.80mm_HandSolder, F.Cu at (157.9, 143.0)
- added C79: 2.2n, Capacitor_SMD:C_1206_3216Metric_Pad1.33x1.80mm_HandSolder, F.Cu at (157.9, 146.3)
- added C8: 68n, Capacitor_SMD:C_1206_3216Metric_Pad1.33x1.80mm_HandSolder, F.Cu at (115.5, 30.3)
- added C80: 2.2n, Capacitor_SMD:C_1206_3216Metric_Pad1.33x1.80mm_HandSolder, F.Cu at (157.9, 149.7)
- added C81: 2.2n, Capacitor_SMD:C_1206_3216Metric_Pad1.33x1.80mm_HandSolder, F.Cu at (157.9, 153.0)
- added C82: 10u, Capacitor_SMD:C_1206_3216Metric_Pad1.33x1.80mm_HandSolder, F.Cu at (157.9, 156.4)
- added C83: 0.1u, Capacitor_SMD:C_1206_3216Metric_Pad1.33x1.80mm_HandSolder, F.Cu at (163.9, 139.6)
- added C84: 2.2n, Capacitor_SMD:C_1206_3216Metric_Pad1.33x1.80mm_HandSolder, F.Cu at (163.9, 143.0)
- added C85: 10u, Capacitor_SMD:C_1206_3216Metric_Pad1.33x1.80mm_HandSolder, F.Cu at (163.9, 146.3)
- added C86: 0.1u, Capacitor_SMD:C_1206_3216Metric_Pad1.33x1.80mm_HandSolder, F.Cu at (163.9, 149.7)
- added C87: 2.2n, Capacitor_SMD:C_1206_3216Metric_Pad1.33x1.80mm_HandSolder, F.Cu at (163.9, 153.0)
- added C88: 1u, Capacitor_SMD:C_1206_3216Metric_Pad1.33x1.80mm_HandSolder, F.Cu at (163.9, 156.4)
- added C89: 2.2n, Capacitor_SMD:C_1206_3216Metric_Pad1.33x1.80mm_HandSolder, F.Cu at (169.9, 139.6)
- added C9: 10u, Capacitor_SMD:C_1206_3216Metric_Pad1.33x1.80mm_HandSolder, F.Cu at (121.5, 10.2)
- added C90: 10u, Capacitor_SMD:C_1206_3216Metric_Pad1.33x1.80mm_HandSolder, F.Cu at (169.9, 143.0)
- added C91: 0.1u, Capacitor_SMD:C_1206_3216Metric_Pad1.33x1.80mm_HandSolder, F.Cu at (169.9, 146.3)
- added C92: 10u, Capacitor_SMD:C_1206_3216Metric_Pad1.33x1.80mm_HandSolder, F.Cu at (169.9, 149.7)
- added C93: 0.1u, Capacitor_SMD:C_1206_3216Metric_Pad1.33x1.80mm_HandSolder, F.Cu at (169.9, 153.0)
- added C94: 2.2n, Capacitor_SMD:C_1206_3216Metric_Pad1.33x1.80mm_HandSolder, F.Cu at (157.9, 95.4)
- added C95: 2.2n, Capacitor_SMD:C_1206_3216Metric_Pad1.33x1.80mm_HandSolder, F.Cu at (157.9, 98.8)
- added C96: 2.2n, Capacitor_SMD:C_1206_3216Metric_Pad1.33x1.80mm_HandSolder, F.Cu at (157.9, 102.1)
- added C97: 2.2n, Capacitor_SMD:C_1206_3216Metric_Pad1.33x1.80mm_HandSolder, F.Cu at (157.9, 105.5)
- added C98: 2.2n, Capacitor_SMD:C_1206_3216Metric_Pad1.33x1.80mm_HandSolder, F.Cu at (157.9, 108.8)
- added C99: 10u, Capacitor_SMD:C_1206_3216Metric_Pad1.33x1.80mm_HandSolder, F.Cu at (157.9, 112.2)
- added D1: SS34, SS34:DIOM7959X265N, F.Cu at (97.9, 60.2)
- added D10: 1N4004, Diode_THT:D_DO-41_SOD81_P10.16mm_Horizontal, F.Cu at (153.3, 10.6)
- added D11: 1N4004, Diode_THT:D_DO-41_SOD81_P10.16mm_Horizontal, F.Cu at (153.3, 14.9)
- added D12: 1N4004, Diode_THT:D_DO-41_SOD81_P10.16mm_Horizontal, F.Cu at (153.3, 19.1)
- added D13: 1N4004, Diode_THT:D_DO-41_SOD81_P10.16mm_Horizontal, F.Cu at (153.3, 23.4)
- added D14: 1N4004, Diode_THT:D_DO-41_SOD81_P10.16mm_Horizontal, F.Cu at (153.3, 62.4)
- added D15: 1N4004, Diode_THT:D_DO-41_SOD81_P10.16mm_Horizontal, F.Cu at (153.3, 66.7)
- added D16: 1N4004, Diode_THT:D_DO-41_SOD81_P10.16mm_Horizontal, F.Cu at (153.3, 70.9)
- added D17: 1N4004, Diode_THT:D_DO-41_SOD81_P10.16mm_Horizontal, F.Cu at (153.3, 75.2)
- added D18: 1N4004, Diode_THT:D_DO-41_SOD81_P10.16mm_Horizontal, F.Cu at (114.3, 67.1)
- added D19: 1N4004, Diode_THT:D_DO-41_SOD81_P10.16mm_Horizontal, F.Cu at (114.3, 71.4)
- added D2: SS34, SS34:DIOM7959X265N, F.Cu at (97.9, 67.7)
- added D20: 1N4004, Diode_THT:D_DO-41_SOD81_P10.16mm_Horizontal, F.Cu at (114.3, 75.6)
- added D21: 1N4004, Diode_THT:D_DO-41_SOD81_P10.16mm_Horizontal, F.Cu at (114.3, 79.9)
- added D22: BAT54S, Package_TO_SOT_SMD:SOT-23, F.Cu at (51.6, 129.5)
- added D23: BAT54S, Package_TO_SOT_SMD:SOT-23, F.Cu at (51.6, 133.9)
- added D24: BAT54S, Package_TO_SOT_SMD:SOT-23, F.Cu at (51.6, 138.4)
- added D25: BAT54S, Package_TO_SOT_SMD:SOT-23, F.Cu at (51.6, 142.8)
- added D26: BAT54S, Package_TO_SOT_SMD:SOT-23, F.Cu at (51.6, 147.3)
- added D27: BAT54S, Package_TO_SOT_SMD:SOT-23, F.Cu at (51.6, 151.7)
- added D28: BAT54S, Package_TO_SOT_SMD:SOT-23, F.Cu at (51.6, 156.2)
- added D29: BAT54S, Package_TO_SOT_SMD:SOT-23, F.Cu at (56.5, 129.5)
- added D3: SS2PH10, SS2PH10:DO-220AA_SS2PH10-M3&slash_84A_VIS, F.Cu at (146.6, 52.9)
- added D30: BAT54S, Package_TO_SOT_SMD:SOT-23, F.Cu at (56.5, 133.9)
- added D31: BAT54S, Package_TO_SOT_SMD:SOT-23, F.Cu at (56.5, 138.4)
- added D32: BAT54S, Package_TO_SOT_SMD:SOT-23, F.Cu at (56.5, 142.8)
- added D33: BAT54S, Package_TO_SOT_SMD:SOT-23, F.Cu at (56.5, 147.3)
- added D34: BAT54S, Package_TO_SOT_SMD:SOT-23, F.Cu at (56.5, 151.7)
- added D35: BAT54S, Package_TO_SOT_SMD:SOT-23, F.Cu at (56.5, 156.2)
- added D36: BAT54S, Package_TO_SOT_SMD:SOT-23, F.Cu at (61.4, 129.5)
- added D37: BAT54S, Package_TO_SOT_SMD:SOT-23, F.Cu at (61.4, 133.9)
- added D38: BAT54S, Package_TO_SOT_SMD:SOT-23, F.Cu at (61.4, 138.4)
- added D39: BAT54S, Package_TO_SOT_SMD:SOT-23, F.Cu at (61.4, 142.8)
- added D4: B0540W, B0540W:SOD123_DIO-M, F.Cu at (137.8, 51.6)
- added D40: BAT54S, Package_TO_SOT_SMD:SOT-23, F.Cu at (61.4, 147.3)
- added D41: BAT54S, Package_TO_SOT_SMD:SOT-23, F.Cu at (61.4, 151.7)
- added D42: BAT54S, Package_TO_SOT_SMD:SOT-23, F.Cu at (61.4, 156.2)
- added D43: BAT54S, Package_TO_SOT_SMD:SOT-23, F.Cu at (66.3, 129.5)
- added D44: BAT54S, Package_TO_SOT_SMD:SOT-23, F.Cu at (66.3, 133.9)
- added D45: BAT54S, Package_TO_SOT_SMD:SOT-23, F.Cu at (66.3, 138.4)
- added D46: BAT54S, Package_TO_SOT_SMD:SOT-23, F.Cu at (66.3, 142.8)
- added D47: BAT54S, Package_TO_SOT_SMD:SOT-23, F.Cu at (66.3, 147.3)
- added D48: BAT54S, Package_TO_SOT_SMD:SOT-23, F.Cu at (66.3, 151.7)
- added D49: BAT54S, Package_TO_SOT_SMD:SOT-23, F.Cu at (66.3, 156.2)
- added D5: B0540W, B0540W:SOD123_DIO-M, F.Cu at (137.8, 55.1)
- added D50: BAT54S, Package_TO_SOT_SMD:SOT-23, F.Cu at (71.2, 129.5)
- added D51: BAT54S, Package_TO_SOT_SMD:SOT-23, F.Cu at (71.2, 133.9)
- added D52: BAT54S, Package_TO_SOT_SMD:SOT-23, F.Cu at (71.2, 138.4)
- added D53: BAT54S, Package_TO_SOT_SMD:SOT-23, F.Cu at (71.2, 142.8)
- added D54: BAT54S, Package_TO_SOT_SMD:SOT-23, F.Cu at (125.3, 129.5)
- added D55: BAT54S, Package_TO_SOT_SMD:SOT-23, F.Cu at (125.3, 133.9)
- added D56: BAT54S, Package_TO_SOT_SMD:SOT-23, F.Cu at (125.3, 138.4)
- added D57: BAT54S, Package_TO_SOT_SMD:SOT-23, F.Cu at (125.3, 142.8)
- added D58: BAT54S, Package_TO_SOT_SMD:SOT-23, F.Cu at (125.3, 147.3)
- added D59: BAT54S, Package_TO_SOT_SMD:SOT-23, F.Cu at (125.3, 151.7)
- added D6: 1N4004, Diode_THT:D_DO-41_SOD81_P10.16mm_Horizontal, F.Cu at (153.3, 36.5)
- added D60: BAT54S, Package_TO_SOT_SMD:SOT-23, F.Cu at (125.3, 156.2)
- added D61: BAT54S, Package_TO_SOT_SMD:SOT-23, F.Cu at (130.2, 129.5)
- added D62: BAT54S, Package_TO_SOT_SMD:SOT-23, F.Cu at (130.2, 133.9)
- added D63: BAT54S, Package_TO_SOT_SMD:SOT-23, F.Cu at (130.2, 138.4)
- added D64: BAT54S, Package_TO_SOT_SMD:SOT-23, F.Cu at (130.2, 142.8)
- added D65: BAT54S, Package_TO_SOT_SMD:SOT-23, F.Cu at (130.2, 147.3)
- added D66: BAT54S, Package_TO_SOT_SMD:SOT-23, F.Cu at (130.2, 151.7)
- added D67: BAT54S, Package_TO_SOT_SMD:SOT-23, F.Cu at (130.2, 156.2)
- added D68: BAT54S, Package_TO_SOT_SMD:SOT-23, F.Cu at (135.1, 129.5)
- added D69: BAT54S, Package_TO_SOT_SMD:SOT-23, F.Cu at (135.1, 133.9)
- added D7: 1N4004, Diode_THT:D_DO-41_SOD81_P10.16mm_Horizontal, F.Cu at (153.3, 40.8)
- added D70: BAT54S, Package_TO_SOT_SMD:SOT-23, F.Cu at (135.1, 138.4)
- added D71: BAT54S, Package_TO_SOT_SMD:SOT-23, F.Cu at (135.1, 142.8)
- added D72: BAT54S, Package_TO_SOT_SMD:SOT-23, F.Cu at (135.1, 147.3)
- added D73: BAT54S, Package_TO_SOT_SMD:SOT-23, F.Cu at (135.1, 151.7)
- added D74: BAT54S, Package_TO_SOT_SMD:SOT-23, F.Cu at (135.1, 156.2)
- added D75: BAT54S, Package_TO_SOT_SMD:SOT-23, F.Cu at (140.0, 129.5)
- added D76: BAT54S, Package_TO_SOT_SMD:SOT-23, F.Cu at (140.0, 133.9)
- added D77: BAT54S, Package_TO_SOT_SMD:SOT-23, F.Cu at (140.0, 138.4)
- added D78: BAT54S, Package_TO_SOT_SMD:SOT-23, F.Cu at (140.0, 142.8)
- added D79: BAT54S, Package_TO_SOT_SMD:SOT-23, F.Cu at (140.0, 147.3)
- added D8: 1N4004, Diode_THT:D_DO-41_SOD81_P10.16mm_Horizontal, F.Cu at (153.3, 45.0)
- added D80: BAT54S, Package_TO_SOT_SMD:SOT-23, F.Cu at (140.0, 151.7)
- added D81: BAT54S, Package_TO_SOT_SMD:SOT-23, F.Cu at (140.0, 156.2)
- added D82: BAT54S, Package_TO_SOT_SMD:SOT-23, F.Cu at (144.9, 129.5)
- added D83: BAT54S, Package_TO_SOT_SMD:SOT-23, F.Cu at (144.9, 133.9)
- added D84: BAT54S, Package_TO_SOT_SMD:SOT-23, F.Cu at (144.9, 138.4)
- added D85: BAT54S, Package_TO_SOT_SMD:SOT-23, F.Cu at (144.9, 142.8)
- added D9: 1N4004, Diode_THT:D_DO-41_SOD81_P10.16mm_Horizontal, F.Cu at (153.3, 49.3)
- added FB1: FerriteBead_Small, Inductor_SMD:L_1206_3216Metric_Pad1.22x1.90mm_HandSolder, F.Cu at (115.5, 33.7)
- added FB10: FerriteBead_Small, Inductor_SMD:L_1206_3216Metric_Pad1.22x1.90mm_HandSolder, F.Cu at (115.5, 83.7)
- added FB11: FerriteBead_Small, Inductor_SMD:L_1206_3216Metric_Pad1.22x1.90mm_HandSolder, F.Cu at (115.5, 87.2)
- added FB2: FerriteBead_Small, Inductor_SMD:L_1206_3216Metric_Pad1.22x1.90mm_HandSolder, F.Cu at (115.5, 37.1)
- added FB3: FerriteBead_Small, Inductor_SMD:L_1206_3216Metric_Pad1.22x1.90mm_HandSolder, F.Cu at (115.5, 40.6)
- added FB4: FerriteBead_Small, Inductor_SMD:L_1206_3216Metric_Pad1.22x1.90mm_HandSolder, F.Cu at (154.5, 53.1)
- added FB5: FerriteBead_Small, Inductor_SMD:L_1206_3216Metric_Pad1.22x1.90mm_HandSolder, F.Cu at (154.5, 56.6)
- added FB6: FerriteBead_Small, Inductor_SMD:L_1206_3216Metric_Pad1.22x1.90mm_HandSolder, F.Cu at (154.5, 27.2)
- added FB7: FerriteBead_Small, Inductor_SMD:L_1206_3216Metric_Pad1.22x1.90mm_HandSolder, F.Cu at (154.5, 30.7)
- added FB8: FerriteBead_Small, Inductor_SMD:L_1206_3216Metric_Pad1.22x1.90mm_HandSolder, F.Cu at (154.5, 79.0)
- added FB9: FerriteBead_Small, Inductor_SMD:L_1206_3216Metric_Pad1.22x1.90mm_HandSolder, F.Cu at (154.5, 82.5)
- added H1: MountingHole_Pad, MountingHole:MountingHole_3.2mm_M3_Pad_TopBottom, F.Cu at (82.0, 48.9)
- added H2: MountingHole_Pad, MountingHole:MountingHole_3.2mm_M3_Pad_TopBottom, F.Cu at (82.0, 56.9)
- added H3: MountingHole_Pad, MountingHole:MountingHole_3.2mm_M3_Pad_TopBottom, F.Cu at (82.0, 64.8)
- added H4: MountingHole_Pad, MountingHole:MountingHole_3.2mm_M3_Pad_TopBottom, F.Cu at (82.0, 72.8)
- added J1: B3B-XH-AMLFSN, JST_XH:CONN_B3B-XH-AMLFSN_JST, F.Cu at (35.6, 12.8)
- added J10: B3B-XH-AMLFSN, JST_XH:CONN_B3B-XH-AMLFSN_JST, F.Cu at (48.3, 12.8)
- added J11: B3B-XH-AMLFSN, JST_XH:CONN_B3B-XH-AMLFSN_JST, F.Cu at (48.3, 20.2)
- added J12: B3B-XH-AMLFSN, JST_XH:CONN_B3B-XH-AMLFSN_JST, F.Cu at (48.3, 27.7)
- added J13: B3B-XH-AMLFSN, JST_XH:CONN_B3B-XH-AMLFSN_JST, F.Cu at (48.3, 35.1)
- added J14: B3B-XH-AMLFSN, JST_XH:CONN_B3B-XH-AMLFSN_JST, F.Cu at (48.3, 42.6)
- added J15: B3B-XH-AMLFSN, JST_XH:CONN_B3B-XH-AMLFSN_JST, F.Cu at (48.3, 50.0)
- added J16: B3B-XH-AMLFSN, JST_XH:CONN_B3B-XH-AMLFSN_JST, F.Cu at (48.3, 57.5)
- added J17: B3B-XH-AMLFSN, JST_XH:CONN_B3B-XH-AMLFSN_JST, F.Cu at (48.3, 64.9)
- added J18: B3B-XH-AMLFSN, JST_XH:CONN_B3B-XH-AMLFSN_JST, F.Cu at (48.3, 72.4)
- added J19: B3B-XH-AMLFSN, JST_XH:CONN_B3B-XH-AMLFSN_JST, F.Cu at (61.0, 12.8)
- added J2: B3B-XH-AMLFSN, JST_XH:CONN_B3B-XH-AMLFSN_JST, F.Cu at (35.6, 20.2)
- added J20: B3B-XH-AMLFSN, JST_XH:CONN_B3B-XH-AMLFSN_JST, F.Cu at (61.0, 20.2)
- added J21: B3B-XH-AMLFSN, JST_XH:CONN_B3B-XH-AMLFSN_JST, F.Cu at (61.0, 27.7)
- added J22: B3B-XH-AMLFSN, JST_XH:CONN_B3B-XH-AMLFSN_JST, F.Cu at (61.0, 35.1)
- added J23: B3B-XH-AMLFSN, JST_XH:CONN_B3B-XH-AMLFSN_JST, F.Cu at (61.0, 42.6)
- added J24: B3B-XH-AMLFSN, JST_XH:CONN_B3B-XH-AMLFSN_JST, F.Cu at (61.0, 50.0)
- added J25: B3B-XH-AMLFSN, JST_XH:CONN_B3B-XH-AMLFSN_JST, F.Cu at (61.0, 57.5)
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Other:
- board outline added: 173.5 x 187.5 mm
